Commit message: xacro

File: urdf/terrain/terrain.xacro (robot description, xacro)
@@ -4,5 +4,5 @@
     <color rgba="0.02 0.26 0.46 0.6"/>
   </material>
-<xacro:macro name="inertia" params="mass">
+<xacro:macro name="inertial" params="mass">
      <inertial>
       <mass value="${mass}"/>
@@ -25,5 +25,5 @@
       </geometry>
     </collision>
-    <xacro:inertia mass="0.5"/>
+    <xacro:inertial mass="0.5"/>
   </link>
     <joint name="terrain_jnt" type="fixed">
@@ -40,5 +40,5 @@
       <material name="water"/>
     </visual>
-     <xacro:inertia mass="0.5"/>
+     <xacro:inertial mass="0.5"/>
   </link>
   <joint name="surface_jnt" type="fixed">

Commit message: xacro2

File: urdf/terrain/terrain.xacro (robot description, xacro)
@@ -4,5 +4,5 @@
     <color rgba="0.02 0.26 0.46 0.6"/>
   </material>
-<xacro:macro name="inertial" params="mass">
+<xacro:macro name="minert" params="mass">
      <inertial>
       <mass value="${mass}"/>
@@ -25,5 +25,5 @@
       </geometry>
     </collision>
-    <xacro:inertial mass="0.5"/>
+    <xacro:minert mass="0.5"/>
   </link>
     <joint name="terrain_jnt" type="fixed">
@@ -40,5 +40,5 @@
       <material name="water"/>
     </visual>
-     <xacro:inertial mass="0.5"/>
+     <xacro:minert mass="0.5"/>
   </link>
   <joint name="surface_jnt" type="fixed">
